Commit message: Adding complex pipes and a parameter file for springs configuration

File: urdf/PIR-B-ASSY-001-description.xacro (robot description, xacro)
@@ -151,5 +151,5 @@
       xyz="0 0 1" />
     <limit
-      effort="3.5"
+      effort="100"
       velocity="10" />
   </joint>
@@ -485,5 +485,5 @@
       xyz="0 0 -1" />
     <limit
-      effort="3.5"
+      effort="100"
       velocity="10" />
   </joint>

File: urdf/PIR-B-ASSY-001-gazebo.xacro (robot description, xacro)
@@ -1,4 +1,14 @@
 <?xml version="1.0" encoding="utf-8"?>
 <robot xmlns:xacro="http://wiki.ros.org/xacro" name="pir-b-001">
+<xacro:property name="_pi" value="3.14159"/>
+<!-- Retrieve parameters from the ROS parameter server -->
+<xacro:property name="spring_param_file" value="$(find pir-b-001)/config/spring_param.yaml" />
+<xacro:property name="spring" value="${xacro.load_yaml(spring_param_file)}"/>
+<xacro:property name="right_linkj_spring_stiffness" value="${spring['right_linkj']['spring_stiffness']}" />
+<xacro:property name="right_linkj_spring_reference" value="${spring['right_linkj']['spring_reference']}" />
+<xacro:property name="left_linkj_spring_stiffness" value="${spring['left_linkj']['spring_stiffness']}" />
+<xacro:property name="left_linkj_spring_reference" value="${spring['left_linkj']['spring_reference']}" />
+<xacro:property name="link3j_spring_stiffness" value="${spring['link3j']['spring_stiffness']}" />
+<xacro:property name="link3j_spring_reference" value="${spring['link3j']['spring_reference']}" />
 <!-- joints transmissions -->
 <transmission name="right_wheel1j_trans">
@@ -65,7 +75,7 @@
 <gazebo reference="right_Linkj">
   <implicitSpringDamper>true</implicitSpringDamper>
-  <springStiffness>1</springStiffness>
-  <springReference>0.0</springReference>
-  <damping>0.2</damping>
+  <springStiffness>${right_linkj_spring_stiffness}</springStiffness>
+  <springReference>${right_linkj_spring_reference * _pi / 180}</springReference>
+  <damping>0.5</damping>
   <kp value="60.0" />
   <kd value="0.0" />
@@ -73,7 +83,7 @@
 <gazebo reference="left_Linkj">
   <implicitSpringDamper>true</implicitSpringDamper>
-  <springStiffness>1</springStiffness>
-  <springReference>0.0</springReference>
-  <damping>0.2</damping>
+  <springStiffness>${left_linkj_spring_stiffness}</springStiffness>
+  <springReference>${left_linkj_spring_reference * _pi / 180}</springReference>
+  <damping>0.5</damping>
   <kp value="60.0" />
   <kd value="0.0" />
@@ -81,7 +91,7 @@
 <gazebo reference="link3j">
   <implicitSpringDamper>true</implicitSpringDamper>
-  <springStiffness>1</springStiffness>
-  <springReference>0.0</springReference>
-  <damping>0.2</damping>
+  <springStiffness>${link3j_spring_stiffness}</springStiffness>
+  <springReference>${link3j_spring_reference * _pi / 180}</springReference>
+  <damping>0.5</damping>
   <kp value="60.0" />
   <kd value="0.0" />
@@ -143,20 +153,4 @@
   <material>Gazebo/YellowGlow</material>
 </gazebo>
-<!-- <gazebo>
-  <plugin name="skid_steer_drive_controller" filename="libgazebo_ros_skid_steer_drive.so">
-    <updateRate>100.0</updateRate>
-    <robotNamespace>/pir_b_001</robotNamespace>
-    <leftFrontJoint>omni3j</leftFrontJoint>
-    <rightFrontJoint>omni33j</rightFrontJoint>
-    <leftRearJoint>omni1j</leftRearJoint>
-    <rightRearJoint>omni11j</rightRearJoint>
-    <wheelSeparation>0.09</wheelSeparation>
-    <wheelDiameter>0.1</wheelDiameter>
-    <robotBaseFrame>base_link</robotBaseFrame>
-    <torque>50</torque>
-    <topicName>/cmd_vel</topicName>
-    <broadcastTF>true</broadcastTF>
-  </plugin>
-</gazebo>  -->
   <!-- Camera Sensor -->
   <gazebo reference="camera_link">

Commit message: fixed a bug

File: urdf/PIR-B-ASSY-001-description.xacro (robot description, xacro)
@@ -86,5 +86,5 @@
   <joint
     name="right_Linkj"
-    type="revolute">
+    type="continuous">
     <origin
       xyz="-0.0014878 0.0595 0"
@@ -95,6 +95,6 @@
       link="right_Link" />
     <axis
-      xyz="1 0 0" />
-      <limit lower="-1.57" upper="1.57" effort="100" velocity="10"/>
+      xyz="-1 0 0" />
+      <limit effort="10" velocity="10"/>
   </joint>
   <link
@@ -366,5 +366,5 @@
   <joint
     name="left_Linkj"
-    type="revolute">
+    type="continuous">
     <origin
       xyz="0.0109878 -0.0625 0"
@@ -376,5 +376,5 @@
     <axis
       xyz="1 0 0" />
-      <limit lower="-1.57" upper="1.57" effort="100" velocity="10"/>
+      <limit effort="10" velocity="10"/>
   </joint>
   <link
@@ -420,5 +420,5 @@
   <joint
     name="link3j"
-    type="revolute">
+    type="continuous">
     <origin
       xyz="0.0044878 0 0.122"
@@ -429,6 +429,6 @@
       link="link3" />
     <axis
-      xyz="-1 0 0" />
-    <limit lower="-1.57" upper="1.57" effort="100" velocity="10"/>
+      xyz="1 0 0" />
+    <limit effort="10" velocity="10"/>
   </joint>
   <link

File: urdf/PIR-B-ASSY-001-gazebo.xacro (robot description, xacro)
@@ -74,26 +74,26 @@
 <!-- Torsional Springs -->
 <gazebo reference="right_Linkj">
-  <implicitSpringDamper>true</implicitSpringDamper>
+  <!-- <implicitSpringDamper>true</implicitSpringDamper>
+  <erp>0.2</erp>
+  <cfm>0.01</cfm> -->
   <springStiffness>${right_linkj_spring_stiffness}</springStiffness>
   <springReference>${right_linkj_spring_reference * _pi / 180}</springReference>
-  <damping>0.5</damping>
-  <kp value="60.0" />
-  <kd value="0.0" />
+  <damping>10.0</damping>
 </gazebo>
 <gazebo reference="left_Linkj">
-  <implicitSpringDamper>true</implicitSpringDamper>
+  <!-- <implicitSpringDamper>true</implicitSpringDamper>
+  <erp>0.2</erp>
+  <cfm>0.01</cfm> -->
   <springStiffness>${left_linkj_spring_stiffness}</springStiffness>
   <springReference>${left_linkj_spring_reference * _pi / 180}</springReference>
-  <damping>0.5</damping>
-  <kp value="60.0" />
-  <kd value="0.0" />
+  <damping>10.0</damping>
 </gazebo>
 <gazebo reference="link3j">
-  <implicitSpringDamper>true</implicitSpringDamper>
+  <!-- <implicitSpringDamper>true</implicitSpringDamper>
+  <erp>0.2</erp>
+  <cfm>0.01</cfm> -->
   <springStiffness>${link3j_spring_stiffness}</springStiffness>
   <springReference>${link3j_spring_reference * _pi / 180}</springReference>
-  <damping>0.5</damping>
-  <kp value="60.0" />
-  <kd value="0.0" />
+  <damping>10.0</damping>
 </gazebo>
 <!-- Links on Gazebo -->
@@ -140,13 +140,17 @@
 <gazebo reference="right_Link">
   <material>Gazebo/ZincYellow</material>
+  <!-- <dampingFactor>0.1</dampingFactor> -->
 </gazebo>
 <gazebo reference="left_Link">
   <material>Gazebo/ZincYellow</material>
+  <!-- <dampingFactor>0.1</dampingFactor> -->
 </gazebo>
 <gazebo reference="link3">
   <material>Gazebo/ZincYellow</material>
+  <!-- <dampingFactor>0.1</dampingFactor> -->
 </gazebo>
 <gazebo reference="base_link">
   <material>Gazebo/ZincYellow</material>
+  <!-- <dampingFactor>0.1</dampingFactor> -->
 </gazebo>
 <gazebo reference="camera_link">

File: urdf/camera.xacro (robot description, xacro)
@@ -4,6 +4,6 @@
         <inertial>
             <origin xyz="0 0 0" rpy="0 0 0"/>
-            <mass value="0.1"/>
-            <inertia ixx="0.001" ixy="0.0" ixz="0.0" iyy="0.001" iyz="0.0" izz="0.001"/>
+            <mass value="0.01"/>
+            <inertia ixx="0.0001" ixy="0.0" ixz="0.0" iyy="0.001" iyz="0.0" izz="0.0001"/>
         </inertial>
         <visual>

Commit message: Finalized submission

File: urdf/PIR-B-ASSY-001-description.xacro (robot description, xacro)
@@ -265,6 +265,6 @@
       xyz="-1 0 0" />
     <limit
-      effort="3.5"
-      velocity="10" />
+      effort="10"
+      velocity="100" />
   </joint>
   <link
@@ -321,6 +321,6 @@
       xyz="-1 0 0" />
     <limit
-      effort="3.5"
-      velocity="10" />
+      effort="10"
+      velocity="100" />
   </joint>
   <link
@@ -599,6 +599,6 @@
       xyz="-1 0 0" />
     <limit
-      effort="3.5"
-      velocity="10" />
+      effort="10"
+      velocity="100" />
   </joint>
   <link
@@ -655,6 +655,6 @@
       xyz="-1 0 0" />
     <limit
-      effort="3.5"
-      velocity="10" />
+      effort="10"
+      velocity="100" />
   </joint>
   <link
@@ -711,6 +711,6 @@
       xyz="1 0 0" />
     <limit
-      effort="3.5"
-      velocity="10" />
+      effort="10"
+      velocity="100" />
   </joint>
   <link
@@ -767,6 +767,6 @@
       xyz="1 0 0" />
     <limit
-      effort="3.5"
-      velocity="10" />
+      effort="10"
+      velocity="100" />
   </joint>
 </pir-b-001>

File: urdf/complex_pipe.urdf (robot description, URDF)
Before this commit: robot complex_pipe, 1 links, 0 joints
Links:
- removed link pipe_link
- added link complex_pipe_link, mass 63.1313238293648; collision mesh filename=package://pir-b-001/meshes/complex_pipe_link.STL; visual mesh filename=package://pir-b-001/meshes/complex_pipe_link.STL

Commit message: phase 2.1 update

File: urdf/PIR-B-ASSY-001-description.xacro (robot description, xacro)
@@ -1,4 +1,8 @@
 <?xml version="1.0" encoding="utf-8"?>
 <pir-b-001 xmlns:xacro="http://wiki.ros.org/xacro" name="pir-b-001">
+  <xacro:property name="rolling_effort_val" value="10" />
+  <xacro:property name="rolling_velocity_val" value="50" />
+  <xacro:property name="driving_effort_val" value="10" />
+  <xacro:property name="driving_velocity_val" value="50" />
   <link name="base_footprint" />
   <link
@@ -151,6 +155,6 @@
       xyz="0 0 1" />
     <limit
-      effort="100"
-      velocity="10" />
+      effort="${rolling_effort_val}"
+      velocity="${rolling_velocity_val}" />
   </joint>
   <link
@@ -265,6 +269,6 @@
       xyz="-1 0 0" />
     <limit
-      effort="10"
-      velocity="100" />
+      effort="${driving_effort_val}"
+      velocity="${driving_velocity_val}" />
   </joint>
   <link
@@ -321,6 +325,6 @@
       xyz="-1 0 0" />
     <limit
-      effort="10"
-      velocity="100" />
+      effort="${driving_effort_val}"
+      velocity="${driving_velocity_val}" />
   </joint>
   <link
@@ -485,6 +489,6 @@
       xyz="0 0 -1" />
     <limit
-      effort="100"
-      velocity="10" />
+      effort="${rolling_effort_val}"
+      velocity="${rolling_velocity_val}" />
   </joint>
   <link
@@ -599,6 +603,6 @@
       xyz="-1 0 0" />
     <limit
-      effort="10"
-      velocity="100" />
+      effort="${driving_effort_val}"
+      velocity="${driving_velocity_val}" />
   </joint>
   <link
@@ -655,6 +659,6 @@
       xyz="-1 0 0" />
     <limit
-      effort="10"
-      velocity="100" />
+      effort="${driving_effort_val}"
+      velocity="${driving_velocity_val}" />
   </joint>
   <link
@@ -711,6 +715,6 @@
       xyz="1 0 0" />
     <limit
-      effort="10"
-      velocity="100" />
+      effort="${driving_effort_val}"
+      velocity="${driving_velocity_val}" />
   </joint>
   <link
@@ -767,6 +771,6 @@
       xyz="1 0 0" />
     <limit
-      effort="10"
-      velocity="100" />
+      effort="${driving_effort_val}"
+      velocity="${driving_velocity_val}" />
   </joint>
 </pir-b-001>

File: urdf/PIR-B-ASSY-001-gazebo.xacro (robot description, xacro)
@@ -11,4 +11,9 @@
 <xacro:property name="link3j_spring_stiffness" value="${spring['link3j']['spring_stiffness']}" />
 <xacro:property name="link3j_spring_reference" value="${spring['link3j']['spring_reference']}" />
+<!-- wheel friction coefficient -->
+<xacro:property name="mu1_omni_val" value="0.5" />
+<xacro:property name="mu2_omni_val" value="0.7" />
+<xacro:property name="mu1_hemi_val" value="0.5" />
+<xacro:property name="mu2_hemi_val" value="0.9" />
 <!-- joints transmissions -->
 <transmission name="right_wheel1j_trans">
@@ -79,5 +84,5 @@
   <springStiffness>${right_linkj_spring_stiffness}</springStiffness>
   <springReference>${right_linkj_spring_reference * _pi / 180}</springReference>
-  <damping>10.0</damping>
+  <damping>100000.0</damping>
 </gazebo>
 <gazebo reference="left_Linkj">
@@ -87,5 +92,5 @@
   <springStiffness>${left_linkj_spring_stiffness}</springStiffness>
   <springReference>${left_linkj_spring_reference * _pi / 180}</springReference>
-  <damping>10.0</damping>
+  <damping>100000.0</damping>
 </gazebo>
 <gazebo reference="link3j">
@@ -95,45 +100,45 @@
   <springStiffness>${link3j_spring_stiffness}</springStiffness>
   <springReference>${link3j_spring_reference * _pi / 180}</springReference>
-  <damping>10.0</damping>
+  <damping>100000.0</damping>
 </gazebo>
 <!-- Links on Gazebo -->
 <gazebo reference="omni1">
-  <mu1 value="0.5"/>
-  <mu2 value="0.7"/>
+  <mu1 value="${mu1_omni_val}"/>
+  <mu2 value="${mu2_omni_val}"/>
   <material>Gazebo/Black</material>
 </gazebo>
 <gazebo reference="omni11">
-  <mu1 value="0.5"/>
-  <mu2 value="0.7"/>
+  <mu1 value="${mu1_omni_val}"/>
+  <mu2 value="${mu2_omni_val}"/>
   <material>Gazebo/Black</material>
 </gazebo>
 <gazebo reference="omni3">
-  <mu1 value="0.5"/>
-  <mu2 value="0.7"/>
+  <mu1 value="${mu1_omni_val}"/>
+  <mu2 value="${mu2_omni_val}"/>
   <material>Gazebo/Black</material>
 </gazebo>
 <gazebo reference="omni33">
-  <mu1 value="0.5"/>
-  <mu2 value="0.7"/>
+  <mu1 value="${mu1_omni_val}"/>
+  <mu2 value="${mu2_omni_val}"/>
   <material>Gazebo/Black</material>
 </gazebo>
 <gazebo reference="omni2">
-  <mu1 value="0.5"/>
-  <mu2 value="0.7"/>
+  <mu1 value="${mu1_omni_val}"/>
+  <mu2 value="${mu2_omni_val}"/>
   <material>Gazebo/Black</material>
 </gazebo>
 <gazebo reference="omni22">
-  <mu1 value="0.5"/>
-  <mu2 value="0.7"/>
+  <mu1 value="${mu1_omni_val}"/>
+  <mu2 value="${mu2_omni_val}"/>
   <material>Gazebo/Black</material>
 </gazebo>
 <gazebo reference="right_wheel">
-  <mu1 value="0.5"/>
-  <mu2 value="0.7"/>
+  <mu1 value="${mu1_hemi_val}"/>
+  <mu2 value="${mu2_hemi_val}"/>
   <material>Gazebo/DarkGrey</material>
 </gazebo>
 <gazebo reference="left_wheel">
-  <mu1 value="0.5"/>
-  <mu2 value="0.7"/>
+  <mu1 value="${mu1_hemi_val}"/>
+  <mu2 value="${mu2_hemi_val}"/>
   <material>Gazebo/DarkGrey</material>
 </gazebo>
@@ -154,43 +159,59 @@
   <!-- <dampingFactor>0.1</dampingFactor> -->
 </gazebo>
+<!-- Camera Sensor -->
 <gazebo reference="camera_link">
   <material>Gazebo/YellowGlow</material>
-</gazebo>
-  <!-- Camera Sensor -->
-  <gazebo reference="camera_link">
-    <sensor type="camera" name="camera">
-      <update_rate>30.0</update_rate>
-      <camera name="head">
-        <horizontal_fov>1.3962634</horizontal_fov>
-        <image>
-          <width>800</width>
-          <height>800</height>
-          <format>R8G8B8</format>
-        </image>
-        <clip>
-          <near>0.02</near>
-          <far>300</far>
-        </clip>
-        <noise>
-          <type>gaussian</type>
-          <mean>0.0</mean>
-          <stddev>0.007</stddev>
-        </noise>
-      </camera>
-      <plugin name="camera_controller" filename="libgazebo_ros_camera.so">
-        <alwaysOn>true</alwaysOn>
-        <updateRate>30.0</updateRate>
-        <cameraName>camera</cameraName>
-        <imageTopicName>image_raw</imageTopicName>
-        <cameraInfoTopicName>camera_info</cameraInfoTopicName>
+  <sensor type="camera" name="camera">
+    <update_rate>30.0</update_rate>
+    <camera name="head">
+      <horizontal_fov>1.3962634</horizontal_fov>
+      <image>
+        <width>640</width>
+        <height>480</height>
+        <format>R8G8B8</format>
+      </image>
+      <clip>
+        <near>0.02</near>
+        <far>300</far>
+      </clip>
+      <noise>
+        <type>gaussian</type>
+        <mean>0.0</mean>
+        <stddev>0.007</stddev>
+      </noise>
+    </camera>
+    <plugin name="camera_controller" filename="libgazebo_ros_camera.so">
+      <alwaysOn>true</alwaysOn>
+      <updateRate>30.0</updateRate>
+      <cameraName>camera</cameraName>
+      <imageTopicName>image_raw</imageTopicName>
+      <cameraInfoTopicName>camera_info</cameraInfoTopicName>
+      <frameName>camera_link</frameName>
+      <hackBaseline>0.07</hackBaseline>
+      <distortionK1>0.0</distortionK1>
+      <distortionK2>0.0</distortionK2>
+      <distortionK3>0.0</distortionK3>
+      <distortionT1>0.0</distortionT1>
+      <distortionT2>0.0</distortionT2>
+    </plugin>
+  </sensor>
+  <gravity>true</gravity>
+    <sensor name="imu_sensor" type="imu">
+      <always_on>true</always_on>
+      <update_rate>50</update_rate>
+      <visualize>true</visualize>
+      <topic>__default_topic__</topic>
+      <plugin filename="libgazebo_ros_imu_sensor.so" name="imu_plugin">
+        <topicName>imu</topicName>
+        <bodyName>imu_link</bodyName>
+        <updateRateHZ>10.0</updateRateHZ>
+        <gaussianNoise>0.0</gaussianNoise>
+        <xyzOffset>0 0 0</xyzOffset>
+        <rpyOffset>0 0 0</rpyOffset>
         <frameName>camera_link</frameName>
-        <hackBaseline>0.07</hackBaseline>
-        <distortionK1>0.0</distortionK1>
-        <distortionK2>0.0</distortionK2>
-        <distortionK3>0.0</distortionK3>
-        <distortionT1>0.0</distortionT1>
-        <distortionT2>0.0</distortionT2>
+        <initialOrientationAsReference>false</initialOrientationAsReference>
       </plugin>
+      <pose>0 0 0 0 0 0</pose>
     </sensor>
-  </gazebo>
+</gazebo>
 </robot>

File: urdf/PIR-INTEGERATION.urdf (robot description, URDF)
Before this commit: robot pir-b-001, 15 links, 14 joints
Links:
- added link camera_link, mass 0.01; collision box size=0.01 0.01 0.01; visual box size=0.04 0.02 0.02
Joints:
- added joint camera_joint: type fixed, parent right_Link, child camera_link, origin xyz=-0.0075 0.035 0.05 rpy=0 -1.57079632679 -1.57079632679
- joint left_Linkj: limit lower=0 upper=0 effort=30 velocity=30 -> effort=10 velocity=10
- joint left_wheel1j: limit (none) -> effort=10 velocity=50
- joint link3j: axis -1 0 0 -> 1 0 0; limit lower=0 upper=0 effort=30 velocity=30 -> effort=10 velocity=10
- joint omni11j: axis 1 0 0 -> -1 0 0; limit effort=0 velocity=100 -> effort=10 velocity=50
- joint omni1j: axis 1 0 0 -> -1 0 0; limit effort=0 velocity=100 -> effort=10 velocity=50
- joint omni22j: limit effort=0 velocity=0 -> effort=10 velocity=50
- joint omni2j: limit effort=0 velocity=0 -> effort=10 velocity=50
- joint omni33j: axis 1 0 0 -> -1 0 0; limit effort=0 velocity=0 -> effort=10 velocity=50
- joint omni3j: axis 1 0 0 -> -1 0 0; limit effort=0 velocity=0 -> effort=10 velocity=50
- joint right_Linkj: axis 1 0 0 -> -1 0 0; limit lower=0 upper=0 effort=30 velocity=30 -> effort=10 velocity=10
- joint right_wheel1j: limit (none) -> effort=10 velocity=50

File: urdf/camera.xacro (robot description, xacro)
@@ -16,15 +16,15 @@
             </material>
         </visual>
-        <collision>
+        <!-- <collision>
             <origin xyz="0 0 0" rpy="0 0 0"/>
             <geometry>
-                <box size="0.01 0.01 0.01"/>
+                <box size="0.001 0.001 0.001"/>
             </geometry>
-        </collision>
+        </collision> -->
     </link>
     <joint name="camera_joint" type="fixed">
         <parent link="right_Link"/>
         <child link="camera_link"/>
-        <origin xyz="-0.0075 0.035 0.05" rpy= "0 -1.57079632679 -1.57079632679" />
+        <origin xyz="-0.0075 0.035 0.05" rpy= "0 -2.35619449019 -1.57079632679" />
     </joint>
 </robot>
